File: PCBs/node/node.kicad_pcb (KiCad board)
At the start: 2 copper layers, 61 x 57.2 mm, 10 parts, among them J1 Bat+, J2 GND, J3 5V, SW1 SW_Push, U1 ESP32-DEVKIT-V1, U2 BME280, U3 pm25sensor, U4 lidar

Commit message: changes
Parts:
- moved U2 15.2 mm to (92.1, 104.1), turned to 180 degrees
Connections:
- R1 pad 2: Net-(BT2--) -> GND
Routing:
- net Net-(U1-D21): track 42.6 -> 15.6 mm
- net GND: track 94.5 -> 120.3 mm, vias 0 -> 26
- net +5V: track 93.0 -> 112.4 mm
- net +3.3V: track 48.0 -> 63.3 mm
