File: PCBs/node/node.kicad_sch (KiCad schematic)
At the start: 13 parts, among them J1 Bat+, J2 GND, J3 5V, SW1 SW_Push, U1 ESP32-DEVKIT-V1, U2 BME280, U3 pm25sensor, U4 lidar

Commit message: changes
Changed lines of the file:
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@@
     (stroke (width 0) (type default))
   )
-  (wire (pts (xy 97.79 113.03) (xy 97.79 116.84))
+  (wire (pts (xy 97.79 113.03) (xy 97.79 119.38))
     (stroke (width 0) (type default))
   )
@@
     )
   )
-  (symbol (lib_id "power:GND") (at 97.79 116.84 0) (unit 1)
+  (symbol (lib_id "power:GND") (at 97.79 119.38 0) (unit 1)
     (in_bom yes) (on_board yes) (dnp no)
-    (property "Reference" "#PWR010" (at 97.79 123.19 0)
-      (effects (font (size 1.27 1.27)) hide)
-    )
-    (property "Value" "GND" (at 100.33 116.84 0)
-      (effects (font (size 1.27 1.27)))
-    )
-    (property "Footprint" "" (at 97.79 116.84 0)
-      (effects (font (size 1.27 1.27)) hide)
-    )
-    (property "Datasheet" "" (at 97.79 116.84 0)
-      (effects (font (size 1.27 1.27)) hide)
-    )
+    (property "Reference" "#PWR010" (at 97.79 125.73 0)
+      (effects (font (size 1.27 1.27)) hide)
+    )
+    (property "Value" "GND" (at 100.33 119.38 0)
+      (effects (font (size 1.27 1.27)))
+    )
+    (property "Footprint" "" (at 97.79 119.38 0)
+      (effects (font (size 1.27 1.27)) hide)
+    )
+    (property "Datasheet" "" (at 97.79 119.38 0)
+      (effects (font (size 1.27 1.27)) hide)
+    )

Commit message: changes
Parts:
- added J4: USB_B_Micro, symbol Connector:USB_B_Micro
- added U5: ~, symbol New_Library:BMS
- renumbered BMS_and_STEPDOWN1 to STEPUP1
Connections:
- net GND: now also J4.5 (GND), U5. (Vin)
- net at J1.1 (Pin_1), R2.1: no longer STEPUP1. (GND)
- net at BT1.1 (+): now also BT2.1 (+), U5. (Vin); no longer STEPUP1. (GND)
- net at BT2.2 (-): now also BT1.2 (-), U5. (Vin); no longer STEPUP1. (GND)
- new net: J4.1 (VBUS), U5. (Vin)
- new net: STEPUP1. (GND), U5. (Vin) (x2)
Other:
- moved on the sheet: BT1, BT2, J2, J3

Commit message: Integration hardware (#35)
Parts:
- R2: value 20k -> 10k
Connections:
- net +BATT: now reaches J1.1 (Pin_1), R2.1
- net +BATT: now also STEPUP1. (GND), U5. (Vin)
- net at R1.1, R2.2: now also U1.19 (D34); no longer U1.3 (D15)
- new net: STEPUP1. (GND), U5. (Vin)
Changed lines of the file:
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@@
   (junction (at 35.56 95.25) (diameter 0) (color 0 0 0 0)
   )
+  (junction (at 85.09 92.71) (diameter 0) (color 0 0 0 0)
+  )
   (junction (at 186.69 86.36) (diameter 0) (color 0 0 0 0)
   )
   (junction (at 80.01 110.49) (diameter 0) (color 0 0 0 0)
   )
-  (junction (at 97.79 102.87) (diameter 0) (color 0 0 0 0)
-  )
   (junction (at 80.01 102.87) (diameter 0) (color 0 0 0 0)
   )
@@
   (junction (at 35.56 119.38) (diameter 0) (color 0 0 0 0)
   )
+  (junction (at 49.53 104.14) (diameter 0) (color 0 0 0 0)
+  )
+  (junction (at 97.79 104.14) (diameter 0) (color 0 0 0 0)
+  )
   (wire (pts (xy 76.2 102.87) (xy 80.01 102.87))
     (stroke (width 0) (type default))
   )
+  (wire (pts (xy 97.79 104.14) (xy 97.79 105.41))
+    (stroke (width 0) (type default))
+  )
+  (wire (pts (xy 49.53 104.14) (xy 50.8 104.14))
+    (stroke (width 0) (type default))
+  )
+  (wire (pts (xy 104.14 104.14) (xy 97.79 104.14))
+    (stroke (width 0) (type default))
+  )
   (wire (pts (xy 186.69 64.77) (xy 186.69 86.36))
     (stroke (width 0) (type default))
   )
+  (wire (pts (xy 138.43 107.95) (xy 148.59 107.95))
+    (stroke (width 0) (type default))
+  )
   (wire (pts (xy 153.67 64.77) (xy 154.94 64.77))
     (stroke (width 0) (type default))
@@
     (stroke (width 0) (type default))
   )
-  (wire (pts (xy 97.79 102.87) (xy 97.79 101.6))
-    (stroke (width 0) (type default))
-  )
   (wire (pts (xy 140.97 64.77) (xy 138.43 64.77))
     (stroke (width 0) (type default))
@@
     (stroke (width 0) (type default))
   )
+  (wire (pts (xy 148.59 124.46) (xy 104.14 124.46))
+    (stroke (width 0) (type default))
+  )
+  (wire (pts (xy 49.53 102.87) (xy 49.53 104.14))
+    (stroke (width 0) (type default))
+  )
   (wire (pts (xy 198.12 82.55) (xy 198.12 86.36))
     (stroke (width 0) (type default))
@@
     (stroke (width 0) (type default))
   )
-  (wire (pts (xy 48.26 104.14) (xy 50.8 104.14))
+  (wire (pts (xy 48.26 104.14) (xy 49.53 104.14))
+    (stroke (width 0) (type default))
+  )
+  (wire (pts (xy 104.14 124.46) (xy 104.14 104.14))
     (stroke (width 0) (type default))
   )
@@
     (stroke (width 0) (type default))
   )
+  (wire (pts (xy 148.59 107.95) (xy 148.59 124.46))
+    (stroke (width 0) (type default))
+  )
   (wire (pts (xy 154.94 90.17) (xy 157.48 90.17))
     (stroke (width 0) (type default))
@@
     (stroke (width 0) (type default))
   )
-  (wire (pts (xy 97.79 102.87) (xy 97.79 105.41))
+  (wire (pts (xy 97.79 101.6) (xy 97.79 104.14))
     (stroke (width 0) (type default))
   )
@@
     (stroke (width 0) (type default))
   )
-  (wire (pts (xy 107.95 102.87) (xy 97.79 102.87))
-    (stroke (width 0) (type default))
-  )
   (wire (pts (xy 107.95 119.38) (xy 186.69 119.38))
     (stroke (width 0) (type default))
@@
     (stroke (width 0) (type default))
   )
+  (wire (pts (xy 82.55 92.71) (xy 85.09 92.71))
+    (stroke (width 0) (type default))
+  )
   (wire (pts (xy 104.14 87.63) (xy 107.95 87.63))
     (stroke (width 0) (type default))
@@
       (effects (font (size 1.27 1.27)) (justify left))
     )
-    (property "Value" "20k" (at 100.33 99.06 0)
+    (property "Value" "10k" (at 100.33 99.06 0)
       (effects (font (size 1.27 1.27)) (justify left))
     )
@@
         (path "/e17a9990-ee8f-4c5d-8af3-669130957dbb"
           (reference "U3") (unit 1)
+        )
+      )
+    )
+  )
+  (symbol (lib_id "power:+BATT") (at 49.53 102.87 0) (unit 1)
+    (in_bom yes) (on_board yes) (dnp no) (fields_autoplaced)
+    (property "Reference" "#PWR017" (at 49.53 106.68 0)
+      (effects (font (size 1.27 1.27)) hide)
+    )
+    (property "Value" "+BATT" (at 49.53 97.79 0)
+      (effects (font (size 1.27 1.27)))
+    )
+    (property "Footprint" "" (at 49.53 102.87 0)
+      (effects (font (size 1.27 1.27)) hide)
+    )
+    (property "Datasheet" "" (at 49.53 102.87 0)
+      (effects (font (size 1.27 1.27)) hide)
+    )
+    (pin "1")
+    (instances
+      (project "node"
+        (path "/e17a9990-ee8f-4c5d-8af3-669130957dbb"
+          (reference "#PWR017") (unit 1)
         )
       )
@@
         )
       )
+    )
+  )
+  (symbol (lib_id "power:+BATT") (at 82.55 92.71 90) (unit 1)
+    (in_bom yes) (on_board yes) (dnp no) (fields_autoplaced)
+    (property "Reference" "#PWR016" (at 86.36 92.71 0)
+      (effects (font (size 1.27 1.27)) hide)
+    )
+    (property "Value" "+BATT" (at 78.74 92.71 90)
+      (effects (font (size 1.27 1.27)) (justify left))
+    )
+    (property "Footprint" "" (at 82.55 92.71 0)
+      (effects (font (size 1.27 1.27)) hide)
+    )
+    (property "Datasheet" "" (at 82.55 92.71 0)
+      (effects (font (size 1.27 1.27)) hide)
+    )
+    (pin "1")
+    (instances
+      (project "node"
+        (path "/e17a9990-ee8f-4c5d-8af3-669130957dbb"
+          (reference "#PWR016") (unit 1)
+        )
+      )
