File: PCBs/gateway/gateway.kicad_sch (KiCad schematic)
At the start: 3 parts, among them U1 ESP32-DEVKIT-V1, U2 ESP32-DEVKIT-V1, U4 EA_T123X-I2C

Commit message: changes
Parts:
- added J1: USB_B_Micro, symbol Connector:USB_B_Micro
- added SW1: SW_Push, symbol Switch:SW_Push
- U4: value EA_T123X-I2C -> LCD
Connections:
- net +5V: now also J1.1 (VBUS)
- net GND: now also J1.5 (GND), SW1.1
- net at U2.4 (D2): now also SW1.2
Changed lines of the file:
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@@
+    (stroke (width 0) (type default))
+  )
+  (wire (pts (xy 205.74 78.74) (xy 205.74 81.28))
     (stroke (width 0) (type default))
   )
@@
     (stroke (width 0) (type default))
   )
+  (wire (pts (xy 180.34 99.06) (xy 185.42 99.06))
+    (stroke (width 0) (type default))
+  )
   (wire (pts (xy 147.32 93.98) (xy 147.32 95.25))
     (stroke (width 0) (type default))
@@
     (stroke (width 0) (type default))
   )
+  (wire (pts (xy 196.85 63.5) (xy 196.85 60.96))
+    (stroke (width 0) (type default))
+  )
   (wire (pts (xy 143.51 133.35) (xy 193.04 133.35))
     (stroke (width 0) (type default))
@@
     (stroke (width 0) (type default))
   )
+  (wire (pts (xy 198.12 63.5) (xy 196.85 63.5))
+    (stroke (width 0) (type default))
+  )
   (wire (pts (xy 102.87 73.66) (xy 102.87 76.2))
     (stroke (width 0) (type default))
@@
     (stroke (width 0) (type default))
   )
+  (wire (pts (xy 182.88 88.9) (xy 185.42 88.9))
+    (stroke (width 0) (type default))
+  )
   (wire (pts (xy 185.42 121.92) (xy 180.34 121.92))
     (stroke (width 0) (type default))
   )
+  (symbol (lib_id "power:GND") (at 182.88 88.9 0) (unit 1)
+    (in_bom yes) (on_board yes) (dnp no) (fields_autoplaced)
+    (property "Reference" "#PWR07" (at 182.88 95.25 0)
+      (effects (font (size 1.27 1.27)) hide)
+    )
+    (property "Value" "GND" (at 182.88 93.98 0)
+      (effects (font (size 1.27 1.27)))
+    )
+    (property "Footprint" "" (at 182.88 88.9 0)
+      (effects (font (size 1.27 1.27)) hide)
+    )
+    (property "Datasheet" "" (at 182.88 88.9 0)
+      (effects (font (size 1.27 1.27)) hide)
+    )
+    (pin "1")
+    (instances
+      (project "gateway"
+        (path "/11f12539-b4d8-49b1-aa61-d34776b60659"
+          (reference "#PWR07") (unit 1)
+        )
+      )
+    )
+  )
   (symbol (lib_id "power:GND") (at 149.86 129.54 0) (unit 1)
     (in_bom yes) (on_board yes) (dnp no) (fields_autoplaced)
@@
     )
   )
+  (symbol (lib_id "power:GND") (at 205.74 81.28 0) (unit 1)
+    (in_bom yes) (on_board yes) (dnp no) (fields_autoplaced)
+    (property "Reference" "#PWR08" (at 205.74 87.63 0)
+      (effects (font (size 1.27 1.27)) hide)
+    )
+    (property "Value" "GND" (at 205.74 86.36 0)
+      (effects (font (size 1.27 1.27)))
+    )
+    (property "Footprint" "" (at 205.74 81.28 0)
+      (effects (font (size 1.27 1.27)) hide)
+    )
+    (property "Datasheet" "" (at 205.74 81.28 0)
+      (effects (font (size 1.27 1.27)) hide)
+    )
+    (pin "1")
+    (instances
+      (project "gateway"
+        (path "/11f12539-b4d8-49b1-aa61-d34776b60659"
+          (reference "#PWR08") (unit 1)
+        )
+      )
+    )
+  )
   (symbol (lib_id "power:+5V") (at 102.87 73.66 0) (unit 1)
     (in_bom yes) (on_board yes) (dnp no) (fields_autoplaced)
@@
         (path "/11f12539-b4d8-49b1-aa61-d34776b60659"
           (reference "#PWR01") (unit 1)
+        )
+      )
+    )
+  )
+  (symbol (lib_id "Switch:SW_Push") (at 185.42 93.98 270) (unit 1)
+    (in_bom yes) (on_board yes) (dnp no) (fields_autoplaced)
+    (property "Reference" "SW1" (at 189.23 92.71 90)
+      (effects (font (size 1.27 1.27)) (justify left))
+    )
+    (property "Value" "SW_Push" (at 189.23 95.25 90)
+      (effects (font (size 1.27 1.27)) (justify left))
+    )
+    (property "Footprint" "" (at 190.5 93.98 0)
+      (effects (font (size 1.27 1.27)) hide)
+    )
+    (property "Datasheet" "~" (at 190.5 93.98 0)
+      (effects (font (size 1.27 1.27)) hide)
+    )
+    (pin "1")
+    (pin "2")
+    (instances
+      (project "gateway"
+        (path "/11f12539-b4d8-49b1-aa61-d34776b60659"
+          (reference "SW1") (unit 1)
         )
       )
@@
       (effects (font (size 1.27 1.27)) (justify left))
     )
-    (property "Value" "EA_T123X-I2C" (at 223.52 107.95 0)
+    (property "Value" "LCD" (at 223.52 107.95 0)
       (effects (font (size 1.27 1.27)) (justify left))
     )
@@
         (path "/11f12539-b4d8-49b1-aa61-d34776b60659"
           (reference "U4") (unit 1)
+        )
+      )
+    )
+  )
+  (symbol (lib_id "Connector:USB_B_Micro") (at 205.74 68.58 0) (mirror y) (unit 1)
+    (in_bom yes) (on_board yes) (dnp no)
+    (property "Reference" "J1" (at 205.74 55.88 0)
+      (effects (font (size 1.27 1.27)))
+    )
+    (property "Value" "USB_B_Micro" (at 205.74 58.42 0)
+      (effects (font (size 1.27 1.27)))
+    )
+    (property "Footprint" "" (at 201.93 69.85 0)
+      (effects (font (size 1.27 1.27)) hide)
+    )
+    (property "Datasheet" "~" (at 201.93 69.85 0)
+      (effects (font (size 1.27 1.27)) hide)
+    )
+    (pin "6")
+    (pin "5")
+    (pin "1")
+    (pin "3")
+    (pin "2")
+    (pin "4")
+    (instances
+      (project "gateway"
+        (path "/11f12539-b4d8-49b1-aa61-d34776b60659"
+          (reference "J1") (unit 1)
         )
       )
@@
         )
       )
+    )
+  )
+  (symbol (lib_id "power:+5V") (at 196.85 60.96 0) (unit 1)
+    (in_bom yes) (on_board yes) (dnp no) (fields_autoplaced)
+    (property "Reference" "#PWR09" (at 196.85 64.77 0)
+      (effects (font (size 1.27 1.27)) hide)
+    )
+    (property "Value" "+5V" (at 196.85 55.88 0)
+      (effects (font (size 1.27 1.27)))
+    )
+    (property "Footprint" "" (at 196.85 60.96 0)
+      (effects (font (size 1.27 1.27)) hide)
+    )
+    (property "Datasheet" "" (at 196.85 60.96 0)
+      (effects (font (size 1.27 1.27)) hide)
+    )
+    (pin "1")
+    (instances
+      (project "gateway"
+        (path "/11f12539-b4d8-49b1-aa61-d34776b60659"
+          (reference "#PWR09") (unit 1)
+        )
+      )
